File: FMradio/Fm_radio.kicad_sch (KiCad schematic)
At the start: 68 parts

Commit message: Update
Parts:
- added C7: 47p, Capacitor_THT:C_Disc_D5.0mm_W2.5mm_P5.00mm, symbol mylib:C
- added R28: 100, Resistor_THT:R_Axial_DIN0207_L6.3mm_D2.5mm_P10.16mm_Horizontal, symbol mylib:R
- C17: value 4.7n -> 10n
- C9: value 3.3n -> 10n
- CD1: value BB910 -> BB112
- R23: value 220 -> 680
- VT1, VT6: value 2N3906 -> 2N5401
- VT2: value S9018 -> BF517
Connections:
- net GND: now also C24.2, C7.1; no longer C24.1
- net at C4.1, R10.2, R2.2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: now also R28.1; no longer R1.1, R7.2, R8.2
- net at C22.1, C23.1, R22.1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: now also C24.1; no longer C24.2
- new net: C7.2, R1.1, R28.2, R7.2, R8.2
Other:
- moved on the sheet: AE1, BA1, C1, C10, C11, C12, C17, C18, C2, C22, C3, C4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
